File: HW4/HW4/HW4.kicad_sch (KiCad schematic)
At the start: 22 parts, among them J1 Adafruit CP2102 Friend, J2 Battery, J3 LEFT, J4 RIGHT, SW1 SW_Push, SW2 SW_Push, U2 AP7381-3.3V Linear Regulator

Commit message: HW4 Finish
Parts:
- removed U1: ~, symbol hw4_1:PIC32MX170F256B
- added C6: 1uF, Capacitor_THT:C_Disc_D5.1mm_W3.2mm_P5.00mm, symbol hw4_1:C
- added U3: ~, Package_DIP:DIP-28_W7.62mm_LongPads, symbol hw4_1:PIC32MX170F256B
- C1: value 2.2uF -> 1uF; footprint (none) -> Capacitor_THT:C_Disc_D5.1mm_W3.2mm_P5.00mm
- C2, C4: footprint (none) -> Capacitor_THT:C_Disc_D5.1mm_W3.2mm_P5.00mm
- C3, C5: footprint (none) -> Capacitor_THT:C_Disc_D3.4mm_W2.1mm_P2.50mm
- D1, D2, D3: footprint (none) -> LED_THT:LED_D3.0mm
- J1: footprint (none) -> Connector_PinSocket_2.54mm:PinSocket_1x06_P2.54mm_Vertical
- J2: footprint (none) -> Connector_PinSocket_2.54mm:PinSocket_1x02_P2.54mm_Vertical
- J3, J4: footprint (none) -> Connector_PinSocket_2.54mm:PinSocket_1x12_P2.54mm_Vertical
- R1, R2, R3, R4, R5: footprint (none) -> Resistor_THT:R_Axial_DIN0207_L6.3mm_D2.5mm_P7.62mm_Horizontal
- S2: footprint digikey-footprints:Switch_Slide_11.6x4mm_EG1218 -> pic32board:slideswitch
- SW1, SW2: footprint (none) -> pic32board:push_button
- U2: footprint Package_TO_SOT_THT:TO-92_Inline_Wide -> Package_TO_SOT_THT:TO-92_Inline
Connections:
- net +3.3V: now also U3.13 (VDD), U3.28 (AVDD)
- net A0: now also U3.2 (A0)
- net A1: now also U3.3 (A1)
- net A3: now also U3.10 (A3)
- net A4: now also U3.12 (A4)
- net B0: now also U3.4 (B0)
- net B1: now also U3.5 (B1)
- net B10: now also U3.21 (B10)
- net B11: now also U3.22 (B11)
- net B12: now also U3.23 (B12)
- net B13: now also U3.24 (B13)
- net B14: now also U3.25 (B14)
- net B15: now also U3.26 (B15)
- net B2: now also U3.6 (B2)
- net B6: now also U3.15 (B6)
- net B7: now also U3.16 (B7)
- net B8: now also U3.17 (B8)
- net B9: now also U3.18 (B9)
- net GND: now also C6.2, U3.19 (VSS), U3.27 (AVSS), U3.8 (VSS); no longer C1.2
- net GREEN: now also U3.11 (B4)
- net U1RX: now also U3.9 (A2)
- net U1TX: now also U3.7 (B3)
- net YELLOW: now also U3.14 (B5)
- net at C4.2: now also U3.20 (VCAP)
- net at R5.2, SW2.1: now also U3.1 (~{MCLR})
- new net: C1.2, C6.1
